Commit message: Actualización de códigos MATLAB, software y simulación

File: Hardware/Brazo General/brazo_robotico_urdf/Ensamblee/urdf/Ensamblee.urdf (robot description, URDF)
Before this commit: robot Ensamblee, 7 links, 6 joints
Links:
- added link ensamblaje_corto, mass 0.05; collision mesh filename=model://Ensamblee/meshes/ensamblaje_corto.STL; visual mesh filename=model://Ensamblee/meshes/ensamblaje_corto.STL
- added link world
- link base_giratoria: geometry collision mesh filename=model://Ensamblee/meshes/base_giratoria.STL; visual mesh filename=model://Ensamblee/meshes/base_giratoria.STL
- link base_link: geometry collision mesh filename=model://Ensamblee/meshes/base_link.STL; visual mesh filename=model://Ensamblee/meshes/base_link.STL
- link brazo_inferior: geometry collision mesh filename=model://Ensamblee/meshes/brazo_inferior.STL; visual mesh filename=model://Ensamblee/meshes/brazo_inferior.STL
- link brazo_superior: geometry collision mesh filename=model://Ensamblee/meshes/brazo_superior.STL; visual mesh filename=model://Ensamblee/meshes/brazo_superior.STL
- link dedo_1: mass 0.0045852 -> None; geometry visual mesh filename=model://Ensamblee/meshes/dedo_1.STL
- link dedo_2: mass 0.0045852 -> None; geometry visual mesh filename=model://Ensamblee/meshes/dedo_2.STL
- link dedo_3: mass 0.0045852 -> None; geometry visual mesh filename=model://Ensamblee/meshes/dedo_3.STL
Joints:
- added joint fixed_base: type fixed, parent world, child base_link, origin xyz=0 0 0 rpy=0 0 0
- added joint joint_corto: type fixed, parent brazo_superior, child ensamblaje_corto, origin xyz=0.125 0 0 rpy=0 0 0
- joint joint_4: axis 0 0 -1 -> 0 0 1; origin xyz=0.12475 -0.0039498 -0.0063922 rpy=2.2502 0.079705 0.017371 -> xyz=0.03 -0.01 0.01 rpy=2.25 0 0; parent brazo_superior -> ensamblaje_corto
- joint joint_5: axis 0 0 -1 -> 0 0 1; origin xyz=0.12464 -0.0062567 0.008678 rpy=-1.942 0.065782 -0.072428 -> xyz=0.03 -0.01 -0.01 rpy=-1.94 0 0; parent brazo_superior -> ensamblaje_corto
- joint joint_6: axis 0 0 -1 -> 0 0 1; origin xyz=0.12401 -0.019698 -0.0021097 rpy=0.15313 -0.0049958 -0.015269 -> xyz=0.03 0.02 0 rpy=0.15 0 0; parent brazo_superior -> ensamblaje_corto

File: Simulación/ros2_ws/src/brazo_robotico_urdf/Ensamblee/urdf/Ensamblee.urdf (robot description, URDF)
Before this commit: robot Ensamblee, 8 links, 7 joints
Links:
- added link ensamblaje_corto, mass 0.05; collision mesh filename=model://Ensamblee/meshes/ensamblaje_corto.STL; visual mesh filename=model://Ensamblee/meshes/ensamblaje_corto.STL
- link dedo_1: mass 0.0045852 -> None; geometry visual mesh filename=model://Ensamblee/meshes/dedo_1.STL
- link dedo_2: mass 0.0045852 -> None; geometry visual mesh filename=model://Ensamblee/meshes/dedo_2.STL
- link dedo_3: mass 0.0045852 -> None; geometry visual mesh filename=model://Ensamblee/meshes/dedo_3.STL
Joints:
- added joint joint_corto: type fixed, parent brazo_superior, child ensamblaje_corto, origin xyz=0.125 0 0 rpy=0 0 0
- joint joint_4: axis 0 0 -1 -> 0 0 1; origin xyz=0.12475 -0.0039498 -0.0063922 rpy=2.2502 0.079705 0.017371 -> xyz=0.03 -0.01 0.01 rpy=2.25 0 0; parent brazo_superior -> ensamblaje_corto
- joint joint_5: axis 0 0 -1 -> 0 0 1; origin xyz=0.12464 -0.0062567 0.008678 rpy=-1.942 0.065782 -0.072428 -> xyz=0.03 -0.01 -0.01 rpy=-1.94 0 0; parent brazo_superior -> ensamblaje_corto
- joint joint_6: axis 0 0 -1 -> 0 0 1; origin xyz=0.12401 -0.019698 -0.0021097 rpy=0.15313 -0.0049958 -0.015269 -> xyz=0.03 0.02 0 rpy=0.15 0 0; parent brazo_superior -> ensamblaje_corto
